File: Hardware/Design/Foozle2650.brd (EAGLE design)
At the start: 88.9 x 63.2 mm, 16 parts, among them IC1 ATF16V8, IC2 AT28C64B-15PU, IC3 62256, Y1 MXO45-3C-1M0000

Commit message: Connected A9 to PLD
Connections:
- net A9: now also IC1.11
Routing:
- net A9: track 68.8 -> 98.1 mm, vias 2 -> 5
Changed lines of the file:
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@@
 <wire x1="67.73535" y1="22.3146" x2="68.71395" y2="21.336" width="0.1524" layer="1"/>
 <wire x1="41.91" y1="21.59" x2="42.799" y2="22.479" width="0.1524" layer="1"/>
-<wire x1="42.799" y1="22.479" x2="47" y2="22.479" width="0.1524" layer="1"/>
-<wire x1="47" y1="22.479" x2="47.371" y2="22.479" width="0.1524" layer="1"/>
+<wire x1="42.799" y1="22.479" x2="46.99" y2="22.479" width="0.1524" layer="1"/>
+<wire x1="46.99" y1="22.479" x2="47" y2="22.479" width="0.1524" layer="1"/>
 <wire x1="9" y1="14" x2="8" y2="13" width="0.1524" layer="16"/>
 <wire x1="11" y1="14" x2="9" y2="14" width="0.1524" layer="16"/>
@@
 <wire x1="8" y1="13" x2="7.62" y2="12.7" width="0.1524" layer="16"/>
 <wire x1="41.5" y1="21.5" x2="41.91" y2="21.59" width="0.1524" layer="16"/>
-<wire x1="62.38875" y1="21.336" x2="61.24575" y2="22.479" width="0.1524" layer="1"/>
-<wire x1="61.24575" y1="22.479" x2="47" y2="22.479" width="0.1524" layer="1"/>
+<wire x1="61.24575" y1="22.479" x2="62.38875" y2="21.336" width="0.1524" layer="1"/>
+<wire x1="47" y1="22.479" x2="61.24575" y2="22.479" width="0.1524" layer="1"/>
 </signal>
 <signal name="A0">
@@
 <wire x1="66.92465" y1="35.0146" x2="67.73535" y2="35.0146" width="0.1524" layer="1"/>
 <wire x1="62.38875" y1="34.036" x2="65.94605" y2="34.036" width="0.1524" layer="1"/>
-<wire x1="68.71395" y1="34.036" x2="82.53" y2="34.036" width="0.1524" layer="1"/>
+<wire x1="68.71395" y1="34.036" x2="73.914" y2="34.036" width="0.1524" layer="1"/>
+<wire x1="73.914" y1="34.036" x2="82.53" y2="34.036" width="0.1524" layer="1"/>
 <wire x1="65.94605" y1="34.036" x2="66.92465" y2="35.0146" width="0.1524" layer="1"/>
 <wire x1="67.73535" y1="35.0146" x2="68.71395" y2="34.036" width="0.1524" layer="1"/>
@@
 <wire x1="53.848" y1="34.036" x2="62.38875" y2="34.036" width="0.1524" layer="16"/>
 <wire x1="39.624" y1="46.99" x2="40.513" y2="46.101" width="0.1524" layer="16"/>
+<contactref element="IC1" pad="11"/>
+<wire x1="77.47" y1="60.96" x2="75.565" y2="59.055" width="0.1524" layer="16"/>
+<wire x1="75.565" y1="59.055" x2="73.914" y2="59.055" width="0.1524" layer="16"/>
+<via x="73.914" y="59.055" extent="1-16" drill="0.254"/>
+<wire x1="73.914" y1="59.055" x2="73.914" y2="42.545" width="0.1524" layer="1"/>
+<via x="73.914" y="42.545" extent="1-16" drill="0.254"/>
+<wire x1="73.914" y1="42.545" x2="73.914" y2="34.036" width="0.1524" layer="16"/>
+<via x="73.914" y="34.036" extent="1-16" drill="0.254"/>
 </signal>
 <signal name="!ROMCS">
