File: Hardware/Design/Foozle2650.sch (EAGLE design)
At the start: 16 parts, among them IC1 ATF16V8, IC2 AT28C64B-15PU, IC3 62256, Y1 MXO45-3C-1M0000

Commit message: Connected A9 to PLD
Connections:
- net A9: now also IC1.I9/!OE
Changed lines of the file:
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@@
 <label x="132.08" y="104.14" size="1.016" layer="95"/>
+</segment>
+<segment>
+<pinref part="IC1" gate="G$1" pin="I9/!OE"/>
+<wire x1="243.84" y1="180.34" x2="251.46" y2="180.34" width="0.1524" layer="91"/>
+<label x="246.38" y="180.34" size="1.016" layer="95"/>
 </segment>
 </net>
